File: carte  IHM/carte  IHM.kicad_sch (KiCad schematic)
At the start: 12 parts, among them J1 tirette, J2 UART CP, J3 init, J4 Conn_01x02, U1 XIAO-ESP32-S3-DIP, U2 TFT_320x240

Commit message: v2
Connections:
- net CS (touch): now also U1.3 (GPIO3/D2/A2); no longer U1.6 (GPIO9/D5/I2C_SCL)
- net CS (écran): now also U1.11 (GPIO9/D10/A10/MOSI); no longer U1.9 (GPIO7/D8/A8/SCK)
- net DC: now also U1.6 (GPIO9/D5/I2C_SCL); no longer U1.4 (GPIO4/D3/A3)
- net MOSI: now also U1.2 (GPIO2/DA/A1); no longer U1.3 (GPIO3/D2/A2)
- net SCK: now also U1.4 (GPIO4/D3/A3); no longer U1.2 (GPIO2/DA/A1)
- net TIRETTE: now also U1.10 (GPIO8/D9/A9/MISO); no longer U1.11 (GPIO9/D10/A10/MOSI)
- net init: now also U1.9 (GPIO7/D8/A8/SCK); no longer U1.10 (GPIO8/D9/A9/MISO)
Other:
- moved on the sheet: C5

Commit message: fixes
Parts:
- C5: footprint Capacitor_THT:CP_Radial_D10.0mm_P5.00mm -> Capacitor_THT:CP_Radial_D5.0mm_P2.00mm
Connections:
- net +5V: now also J4.2 (Pin_2); no longer J4.1 (Pin_1)
- net DC: now also U1.5 (GPIO5/D4/I2C_SDA); no longer U1.6 (GPIO9/D5/I2C_SCL)
- net GND: now also J4.1 (Pin_1); no longer J4.2 (Pin_2)
- net RST: now also U1.6 (GPIO9/D5/I2C_SCL); no longer U1.5 (GPIO5/D4/I2C_SDA)
